File: GameOverBase.kicad_pcb (KiCad board)
At the start: 0 parts

Commit message: Adds first draft PCB format
This is only the edge cuts and will be adapted to fit the components
properly later.
Other:
- board outline added: 40 x 25 mm
- copper layers 0 -> 2
Changed lines of the file:
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@@
-(kicad_pcb (version 20210824) (generator pcbnew)
+(kicad_pcb (version 20220308) (generator pcbnew)
+  (general
+    (thickness 1.6)
+  )
+  (paper "A4")
+  (layers
+    (0 "F.Cu" signal "cobre frontal")
+    (31 "B.Cu" signal "Cobre traseira")
+    (32 "B.Adhes" user "Adesivo traseira")
+    (33 "F.Adhes" user "Adesivo frontal")
+    (34 "B.Paste" user "Pasta traseira")
+    (35 "F.Paste" user "Pasta frontal")
+    (36 "B.SilkS" user "Serigrafia traseira")
+    (37 "F.SilkS" user "Serigrafia frontal")
+    (38 "B.Mask" user "Máscara traseira")
+    (39 "F.Mask" user "Máscara frontal")
+    (40 "Dwgs.User" user "Desenhos utilizador")
+    (41 "Cmts.User" user "Comentários")
+    (42 "Eco1.User" user "User.Eco1")
+    (43 "Eco2.User" user "User.Eco2")
+    (44 "Edge.Cuts" user "Cortes contorno")
+    (45 "Margin" user "Margem")
+    (46 "B.CrtYd" user "Pátio traseira")
+    (47 "F.CrtYd" user "Pátio frontal")
+    (48 "B.Fab" user "Fabricação traseira")
+    (49 "F.Fab" user "Fabricação frontal")
+    (50 "User.1" user "Do utilizador 1")
+    (51 "User.2" user "Do utilizador 2")
+    (52 "User.3" user "Do utilizador 3")
+    (53 "User.4" user "Do utilizador 4")
+    (54 "User.5" user "Do utilizador 5")
+    (55 "User.6" user "Do utilizador 6")
+    (56 "User.7" user "Do utilizador 7")
+    (57 "User.8" user "Do utilizador 8")
+    (58 "User.9" user "Do utilizador 9")
+  )
+  (setup
+    (pad_to_mask_clearance 0)
+    (pcbplotparams
+      (layerselection 0x00010fc_ffffffff)
+      (disableapertmacros false)
+      (usegerberextensions false)
+      (usegerberattributes true)
+      (usegerberadvancedattributes true)
+      (creategerberjobfile true)
+      (dashed_line_dash_ratio 12.000000)
+      (dashed_line_gap_ratio 3.000000)
+      (svgprecision 4)
+      (excludeedgelayer true)
+      (plotframeref false)
+      (viasonmask false)
+      (mode 1)
+      (useauxorigin false)
+      (hpglpennumber 1)
+      (hpglpenspeed 20)
+      (hpglpendiameter 15.000000)
+      (dxfpolygonmode true)
+      (dxfimperialunits true)
+      (dxfusepcbnewfont true)
+      (psnegative false)
+      (psa4output false)
+      (plotreference true)
+      (plotvalue true)
+      (plotinvisibletext false)
+      (sketchpadsonfab false)
+      (subtractmaskfromsilk false)
+      (outputformat 1)
+      (mirror false)
+      (drillshape 1)
+      (scaleselection 1)
+      (outputdirectory "")
+    )
+  )
+  (net 0 "")
+  (gr_line (start 123 80) (end 157 80)
+    (stroke (width 0.1) (type default)) (layer "Edge.Cuts"))
+  (gr_line (start 120 102) (end 120 83)
+    (stroke (width 0.1) (type default)) (layer "Edge.Cuts"))
+  (gr_arc (start 160 102) (mid 159.12132 104.12132) (end 157 105)
+    (stroke (width 0.1) (type default)) (layer "Edge.Cuts"))
+  (gr_line (start 157 105) (end 123 105)
+    (stroke (width 0.1) (type default)) (layer "Edge.Cuts"))
+  (gr_arc (start 123 105) (mid 120.87868 104.12132) (end 120 102)
+    (stroke (width 0.1) (type default)) (layer "Edge.Cuts"))
+  (gr_arc (start 120 83) (mid 120.87868 80.87868) (end 123 80)
+    (stroke (width 0.1) (type default)) (layer "Edge.Cuts"))
+  (gr_arc (start 157 80) (mid 159.12132 80.87868) (end 160 83)
+    (stroke (width 0.1) (type default)) (layer "Edge.Cuts"))
+  (gr_line (start 160 83) (end 160 102)
+    (stroke (width 0.1) (type default)) (layer "Edge.Cuts"))
 )
