File: BreakoutBoard/BreakoutBoard/BreakoutBoard.kicad_sch (KiCad schematic)
At the start: 0 parts

Commit message: Adds schematics for addon breakout board
Parts:
- added H1, H2: ~, symbol Mechanical:MountingHole_Pad
- added J1: addon_conn, GameOver:TXGA_FFC05036-24SBD113W5M_1x24_P0.50mm_Horizontal, symbol GameOver:addon_conn
- added J2, J3: Power, symbol Connector_Generic:Conn_02x02_Row_Letter_Last
- added J4: Conn_01x09, symbol Connector_Generic:Conn_01x09
- added J5: Conn_01x10, symbol Connector_Generic:Conn_01x10
Connections:
- new net: J1.10 (IO5), J4.7 (Pin_7)
- new net: J1.11 (IO17), J4.8 (Pin_8)
- new net: J1.14 (IO16), J5.2 (Pin_2)
- new net: J1.15 (IO4), J5.3 (Pin_3)
- new net: J1.16 (IO2), J5.4 (Pin_4)
- new net: J1.17 (IO15), J5.5 (Pin_5)
- new net: J1.19 (IO34), J5.6 (Pin_6)
- new net: J1.20 (IO35), J5.7 (Pin_7)
- new net: J1.21 (IO32), J5.8 (Pin_8)
- new net: J1.22 (IO33), J5.9 (Pin_9)
- new net: J1.3 (IO23), J4.2 (Pin_2)
- new net: J1.4 (IO22), J4.3 (Pin_3)
- new net: J1.5 (IO21), J4.4 (Pin_4)
- new net: J1.6 (IO19), J4.5 (Pin_5)
- new net: J1.9 (IO18), J4.6 (Pin_6)
- new net +3V3: J1.13 (3v3), J1.2 (3v3), J1.24 (3v3), J1.8 (3v3), J2.1a (Pin_1a), J2.1b (Pin_1b), J3.1a (Pin_1a), J3.1b (Pin_1b), J4.1 (Pin_1), J5.1 (Pin_1)
- new net GND: H1.1, H2.1, J1.1 (GND), J1.12 (GND), J1.18 (GND), J1.23 (GND), J1.7 (GND), J2.2a (Pin_2a), J2.2b (Pin_2b), J3.2a (Pin_2a), J3.2b (Pin_2b), J4.9 (Pin_9), J5.10 (Pin_10)
