File: BNO055Sensor/BNO055Sensor.kicad_sch (KiCad schematic)
At the start: 9 parts, among them J1 addon_conn

Commit message: Removes jumper from sensor Vin pin
I tested using the Vin pin and it worked as expected. Having the jumper
there would probably make power delivery much worse. Also, it's easy
enough to bodge this if we get it wrong since it will be sitting on pin
headers.
Parts:
- removed JP?: SolderJumper_3_Bridged12, symbol Jumper:SolderJumper_3_Bridged12
- gave numbers to parts that had none: 5
Connections:
- net +3V3: now also U1.1 (Vin)
- no-connect marks 5 -> 6
Changed lines of the file:
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@@
     (company "Flávio Amieiro")
+  )
+  (junction (at 87.63 71.12) (diameter 0) (color 0 0 0 0)
+  )
+  (junction (at 87.63 124.46) (diameter 0) (color 0 0 0 0)
   )
   (junction (at 227.33 102.87) (diameter 0) (color 0 0 0 0)
@@
   (no_connect (at 93.98 80.01))
   (no_connect (at 93.98 82.55))
+  (no_connect (at 160.02 74.93))
   (wire (pts (xy 149.86 116.84) (xy 154.94 116.84))
     (stroke (width 0) (type default))
@@
     (stroke (width 0) (type default))
   )
-  (wire (pts (xy 153.67 66.04) (xy 153.67 72.39))
-    (stroke (width 0) (type default))
-  )
   (wire (pts (xy 160.02 127) (xy 167.64 127))
     (stroke (width 0) (type default))
   )
-  (wire (pts (xy 160.02 72.39) (xy 163.83 72.39))
-    (stroke (width 0) (type default))
-  )
   (wire (pts (xy 93.98 110.49) (xy 96.52 110.49))
     (stroke (width 0) (type default))
@@
     (stroke (width 0) (type default))
   )
+  (wire (pts (xy 146.05 82.55) (xy 148.59 82.55))
+    (stroke (width 0) (type default))
+  )
+  (wire (pts (xy 93.98 97.79) (xy 96.52 97.79))
+    (stroke (width 0) (type default))
+  )
+  (wire (pts (xy 227.33 102.87) (xy 232.41 102.87))
+    (stroke (width 0) (type default))
+  )
+  (wire (pts (xy 222.25 99.06) (xy 222.25 102.87))
+    (stroke (width 0) (type default))
+  )
+  (wire (pts (xy 160.02 121.92) (xy 167.64 121.92))
+    (stroke (width 0) (type default))
+  )
   (wire (pts (xy 157.48 72.39) (xy 157.48 74.93))
     (stroke (width 0) (type default))
   )
-  (wire (pts (xy 146.05 82.55) (xy 148.59 82.55))
-    (stroke (width 0) (type default))
-  )
-  (wire (pts (xy 93.98 97.79) (xy 96.52 97.79))
-    (stroke (width 0) (type default))
-  )
-  (wire (pts (xy 227.33 102.87) (xy 232.41 102.87))
-    (stroke (width 0) (type default))
-  )
-  (wire (pts (xy 222.25 99.06) (xy 222.25 102.87))
-    (stroke (width 0) (type default))
-  )
-  (wire (pts (xy 160.02 121.92) (xy 167.64 121.92))
-    (stroke (width 0) (type default))
-  )
-  (wire (pts (xy 160.02 74.93) (xy 160.02 72.39))
-    (stroke (width 0) (type default))
-  )
-  (wire (pts (xy 153.67 72.39) (xy 157.48 72.39))
-    (stroke (width 0) (type default))
-  )
-  (wire (pts (xy 158.75 59.69) (xy 158.75 62.23))
-    (stroke (width 0) (type default))
-  )
   (wire (pts (xy 149.86 127) (xy 154.94 127))
-    (stroke (width 0) (type default))
-  )
-  (wire (pts (xy 163.83 72.39) (xy 163.83 66.04))
     (stroke (width 0) (type default))
   )
@@
   (symbol (lib_id "Device:R_Small_US") (at 157.48 127 90) (unit 1)
     (in_bom yes) (on_board yes)
-    (property "Reference" "R?" (id 0) (at 154.94 124.46 90)
+    (property "Reference" "R3" (id 0) (at 154.94 124.46 90)
       (effects (font (size 1.27 1.27)))
     )
@@
   (symbol (lib_id "power:GND") (at 158.75 97.79 0) (unit 1)
     (in_bom yes) (on_board yes) (fields_autoplaced)
-    (property "Reference" "#PWR?" (id 0) (at 158.75 104.14 0)
+    (property "Reference" "#PWR0103" (id 0) (at 158.75 104.14 0)
       (effects (font (size 1.27 1.27)) hide)
     )
@@
   (symbol (lib_id "Device:R_Small_US") (at 157.48 121.92 90) (unit 1)
     (in_bom yes) (on_board yes)
-    (property "Reference" "R?" (id 0) (at 154.94 119.38 90)
+    (property "Reference" "R2" (id 0) (at 154.94 119.38 90)
       (effects (font (size 1.27 1.27)))
     )
@@
     (pin "1")
   )
-  (symbol (lib_id "power:+3V3") (at 158.75 59.69 0) (unit 1)
-    (in_bom yes) (on_board yes) (fields_autoplaced)
-    (property "Reference" "#PWR?" (id 0) (at 158.75 63.5 0)
-      (effects (font (size 1.27 1.27)) hide)
-    )
-    (property "Value" "+3V3" (id 1) (at 158.75 55.88 0)
-      (effects (font (size 1.27 1.27)))
-    )
-    (property "Footprint" "" (id 2) (at 158.75 59.69 0)
-      (effects (font (size 1.27 1.27)) hide)
-    )
-    (property "Datasheet" "" (id 3) (at 158.75 59.69 0)
+  (symbol (lib_id "power:+3V3") (at 157.48 72.39 0) (unit 1)
+    (in_bom yes) (on_board yes) (fields_autoplaced)
+    (property "Reference" "#PWR0105" (id 0) (at 157.48 76.2 0)
+      (effects (font (size 1.27 1.27)) hide)
+    )
+    (property "Value" "+3V3" (id 1) (at 157.48 68.58 0)
+      (effects (font (size 1.27 1.27)))
+    )
+    (property "Footprint" "" (id 2) (at 157.48 72.39 0)
+      (effects (font (size 1.27 1.27)) hide)
+    )
+    (property "Datasheet" "" (id 3) (at 157.48 72.39 0)
+      (effects (font (size 1.27 1.27)) hide)
+    )
+    (pin "1")
+  )
+  (symbol (lib_id "power:PWR_FLAG") (at 87.63 124.46 90) (unit 1)
+    (in_bom yes) (on_board yes) (fields_autoplaced)
+    (property "Reference" "#FLG0102" (id 0) (at 85.725 124.46 0)
+      (effects (font (size 1.27 1.27)) hide)
+    )
+    (property "Value" "PWR_FLAG" (id 1) (at 83.82 125.095 90)
+      (effects (font (size 1.27 1.27)) (justify left))
+    )
+    (property "Footprint" "" (id 2) (at 87.63 124.46 0)
+      (effects (font (size 1.27 1.27)) hide)
+    )
+    (property "Datasheet" "~" (id 3) (at 87.63 124.46 0)
       (effects (font (size 1.27 1.27)) hide)
     )
@@
   (symbol (lib_id "Device:LED_RGBA") (at 172.72 121.92 0) (unit 1)
     (in_bom yes) (on_board yes) (fields_autoplaced)
-    (property "Reference" "D?" (id 0) (at 172.72 109.22 0)
+    (property "Reference" "D1" (id 0) (at 172.72 109.22 0)
       (effects (font (size 1.27 1.27)))
     )
@@
   (symbol (lib_id "GameOver:Adafruit_BNO055_breakout") (at 158.75 85.09 0) (unit 1)
     (in_bom yes) (on_board yes)
-    (property "Reference" "U?" (id 0) (at 163.83 74.93 0)
+    (property "Reference" "U1" (id 0) (at 163.83 74.93 0)
       (effects (font (size 1.27 1.27)) (justify left))
     )
@@
   (symbol (lib_id "power:+3V3") (at 184.15 115.57 0) (unit 1)
     (in_bom yes) (on_board yes) (fields_autoplaced)
-    (property "Reference" "#PWR?" (id 0) (at 184.15 119.38 0)
+    (property "Reference" "#PWR0104" (id 0) (at 184.15 119.38 0)
       (effects (font (size 1.27 1.27)) hide)
     )
@@
     (pin "1")
   )
-  (symbol (lib_id "Jumper:SolderJumper_3_Bridged12") (at 158.75 66.04 0) (mirror x) (unit 1)
-    (in_bom yes) (on_board yes)
-    (property "Reference" "JP?" (id 0) (at 156.21 63.5 0)
-      (effects (font (size 1.27 1.27)))
-    )
-    (property "Value" "SolderJumper_3_Bridged12" (id 1) (at 158.75 68.834 0)
-      (effects (font (size 1.27 1.27)))
-    )
-    (property "Footprint" "" (id 2) (at 158.75 66.04 0)
-      (effects (font (size 1.27 1.27)) hide)
-    )
-    (property "Datasheet" "~" (id 3) (at 158.75 66.04 0)
-      (effects (font (size 1.27 1.27)) hide)
-    )
-    (pin "1")
-    (pin "2")
-    (pin "3")
+  (symbol (lib_id "power:PWR_FLAG") (at 87.63 71.12 90) (unit 1)
+    (in_bom yes) (on_board yes) (fields_autoplaced)
+    (property "Reference" "#FLG0101" (id 0) (at 85.725 71.12 0)
+      (effects (font (size 1.27 1.27)) hide)
+    )
+    (property "Value" "PWR_FLAG" (id 1) (at 83.82 71.755 90)
+      (effects (font (size 1.27 1.27)) (justify left))
+    )
+    (property "Footprint" "" (id 2) (at 87.63 71.12 0)
+      (effects (font (size 1.27 1.27)) hide)
+    )
+    (property "Datasheet" "~" (id 3) (at 87.63 71.12 0)
+      (effects (font (size 1.27 1.27)) hide)
+    )
+    (pin "1")
   )
   (symbol (lib_id "Device:R_Small_US") (at 157.48 116.84 90) (unit 1)
     (in_bom yes) (on_board yes)
-    (property "Reference" "R?" (id 0) (at 154.94 114.3 90)
+    (property "Reference" "R1" (id 0) (at 154.94 114.3 90)
       (effects (font (size 1.27 1.27)))
     )
@@
   )
   (symbol_instances
+    (path "/d571b8d7-197d-471e-9a0e-569811612b45"
+      (reference "#FLG0101") (unit 1) (value "PWR_FLAG") (footprint "")
+    )
+    (path "/7dba0f7e-d3fc-4882-ab39-7cb63098078b"
+      (reference "#FLG0102") (unit 1) (value "PWR_FLAG") (footprint "")
+    )
     (path "/9688e065-eefa-4bd4-b63c-6f941775746e"
       (reference "#PWR01") (unit 1) (value "GND") (footprint "")
@@
     )
     (path "/451b7b0c-2389-42d4-aee4-1047fc4e3956"
-      (reference "#PWR?") (unit 1) (value "GND") (footprint "")
+      (reference "#PWR0103") (unit 1) (value "GND") (footprint "")
+    )
+    (path "/b9812d32-4417-4322-9afc-f47b11a58fc8"
+      (reference "#PWR0104") (unit 1) (value "+3V3") (footprint "")
     )
     (path "/753b6a30-0b1f-4a06-8b11-d7071636d2b9"
-      (reference "#PWR?") (unit 1) (value "+3V3") (footprint "")
-    )
-    (path "/b9812d32-4417-4322-9afc-f47b11a58fc8"
-      (reference "#PWR?") (unit 1) (value "+3V3") (footprint "")
+      (reference "#PWR0105") (unit 1) (value "+3V3") (footprint "")
     )
     (path "/8e1de14e-ffef-41a5-93e5-703a7302bc9f"
-      (reference "D?") (unit 1) (value "LED_RGBA") (footprint "")
+      (reference "D1") (unit 1) (value "LED_RGBA") (footprint "")
     )
     (path "/72b8070d-6360-4ae2-9e52-c57614a73147"
@@
       (reference "J1") (unit 1) (value "addon_conn") (footprint "GameOver:TXGA_FFC05036-24SBD113W5M_1x24_P0.50mm_Horizontal")
     )
-    (path "/cfc8d50c-9659-46eb-a01a-0c07c13d5803"
-      (reference "JP?") (unit 1) (value "SolderJumper_3_Bridged12") (footprint "")
+    (path "/df729cdb-2037-48dc-ae33-70081f93ee69"
+      (reference "R1") (unit 1) (value "1kΩ") (footprint "")
+    )
+    (path "/714ed8ba-61ed-4362-bd7a-70a8dca07984"
+      (reference "R2") (unit 1) (value "1kΩ") (footprint "")
     )
     (path "/231ff0c9-3fc3-43df-915e-0f8070070eb8"
-      (reference "R?") (unit 1) (value "1kΩ") (footprint "")
-    )
-    (path "/714ed8ba-61ed-4362-bd7a-70a8dca07984"
-      (reference "R?") (unit 1) (value "1kΩ") (footprint "")
-    )
-    (path "/df729cdb-2037-48dc-ae33-70081f93ee69"
-      (reference "R?") (unit 1) (value "1kΩ") (footprint "")
+      (reference "R3") (unit 1) (value "1kΩ") (footprint "")
     )
     (path "/a9369305-45f6-4583-af09-8897bb64b91f"
-      (reference "U?") (unit 1) (value "Adafruit_BNO055_breakout") (footprint "GameOver:Adafruit_BNO055_breakout")
-    )
-  )
+      (reference "U1") (unit 1) (value "Adafruit_BNO055_breakout") (footprint "GameOver:Adafruit_BNO055_breakout")
+    )
+  )
