File: Keypad/Keypad.kicad_pcb (KiCad board)
At the start: 2 copper layers, 50 x 35 mm, 17 parts, among them J1 locked, SW1 TL1240GQ1JCLR, SW2 TL1240GQ1JCLR, SW3 TL1240GQ1JCLR, SW4 TL1240GQ1JCLR, SW5 TL1240GQ1JCLR, SW6 TL1240GQ1JCLR

Commit message: Adds JLCPCB order number placeholder to the Keypad pcb
Other:
- board text added: "JLCJLCJLCJLC"
Changed lines of the file:
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@@
   (gr_arc locked (start 167 80) (mid 169.12132 80.87868) (end 170 83)
     (stroke (width 0.1) (type default)) (layer "Edge.Cuts"))
+  (gr_text "JLCJLCJLCJLC" (at 166.5 100 90) (layer "B.SilkS")
+    (effects (font (size 1 1) (thickness 0.15)) (justify mirror))
+  )
   (via (at 161 100) (size 0.8) (drill 0.4) (layers "F.Cu" "B.Cu") (net 1))
   (via (at 165 105.4) (size 0.8) (drill 0.4) (layers "F.Cu" "B.Cu") (net 1))
