File: Keypad/Keypad.kicad_sch (KiCad schematic)
At the start: 16 parts, among them J1 addon_conn, SW1 TL1240GQ1JCLR, SW2 TL1240GQ1JCLR, SW3 TL1240GQ1JCLR, SW4 TL1240GQ1JCLR, SW5 TL1240GQ1JCLR, SW6 TL1240GQ1JCLR

Commit message: Updates all schematic PDFs to version 1.0
Parts:
- ?: renamed from SW1; value TL1240GQ1JCLR -> (none); footprint GameOver:TL1240GQ1JCLR -> (none)
- ?: renamed from R3; value 100Ω -> (none); footprint Resistor_SMD:R_0805_2012Metric_Pad1.20x1.40mm_HandSolder -> (none)
- ?: renamed from R6; value 100Ω -> (none); footprint Resistor_SMD:R_0805_2012Metric_Pad1.20x1.40mm_HandSolder -> (none)
- ?: renamed from H2; value ~ -> (none); footprint MountingHole:MountingHole_2.2mm_M2_Pad_Via -> (none)
- ?: renamed from SW4; value TL1240GQ1JCLR -> (none); footprint GameOver:TL1240GQ1JCLR -> (none)
- ?: renamed from H1; value ~ -> (none); footprint MountingHole:MountingHole_2.2mm_M2_Pad_Via -> (none)
- ?: renamed from SW5; value TL1240GQ1JCLR -> (none); footprint GameOver:TL1240GQ1JCLR -> (none)
- ?: renamed from LOGO1; value GameOver_logo -> (none); footprint GameOver:logo_fcu -> (none)
- ?: renamed from SW3; value TL1240GQ1JCLR -> (none); footprint GameOver:TL1240GQ1JCLR -> (none)
- ?: renamed from J1; value addon_conn -> (none); footprint GameOver:Addon_conn_TXGA_FFC05036-24SBD113W5M_1x24_P0.50mm_Horizontal -> (none)
- ?: renamed from SW6; value TL1240GQ1JCLR -> (none); footprint GameOver:TL1240GQ1JCLR -> (none)
- ?: renamed from R1; value 100Ω -> (none); footprint Resistor_SMD:R_0805_2012Metric_Pad1.20x1.40mm_HandSolder -> (none)
- ?: renamed from R2; value 100Ω -> (none); footprint Resistor_SMD:R_0805_2012Metric_Pad1.20x1.40mm_HandSolder -> (none)
- ?: renamed from SW2; value TL1240GQ1JCLR -> (none); footprint GameOver:TL1240GQ1JCLR -> (none)
- ?: renamed from R5; value 100Ω -> (none); footprint Resistor_SMD:R_0805_2012Metric_Pad1.20x1.40mm_HandSolder -> (none)
- ?: renamed from R4; value 100Ω -> (none); footprint Resistor_SMD:R_0805_2012Metric_Pad1.20x1.40mm_HandSolder -> (none)
