File: BreakoutBoard/BreakoutBoard.kicad_sch (KiCad schematic)
At the start: 6 parts, among them J1 addon_conn, J2 Power_top, J3 Power_bottom, J4 Conn_01x11, J5 Conn_01x11

Commit message: Updates all schematic PDFs to version 1.0
Parts:
- ?: renamed from J3; value Power_bottom -> (none); footprint Connector_PinHeader_2.54mm:PinHeader_2x02_P2.54mm_Vertical -> (none)
- ?: renamed from LOGO1; value GameOver_logo -> (none); footprint GameOver:logo_fcu -> (none)
- ?: renamed from J2; value Power_top -> (none); footprint Connector_PinHeader_2.54mm:PinHeader_2x02_P2.54mm_Vertical -> (none)
- ?: renamed from J1; value addon_conn -> (none); footprint GameOver:Addon_conn_TXGA_FFC05036-24SBD113W5M_1x24_P0.50mm_Horizontal -> (none)
- ?: renamed from J4; value Conn_01x11 -> (none); footprint Connector_PinHeader_2.54mm:PinHeader_1x11_P2.54mm_Vertical -> (none)
- ?: renamed from J5; value Conn_01x11 -> (none); footprint Connector_PinHeader_2.54mm:PinHeader_1x11_P2.54mm_Vertical -> (none)
